File: framos-csi-adapter.sch (KiCad schematic (older format))
At the start: 41 parts, among them J1 DF40C-60DS-0.4V(51), J2 MSAK24025P30, U1 NTS0102DP, U2 NCP163ASN330T1G

Commit message: Add 3V8 and 1V8 DC/DC to the schematic
Parts:
- removed C3, C6: C_1u_0402, framos-csi-adapter-footprints:0402-cap, symbol framos-csi-adapter:C_1u_0402
- removed C4, C5: C_100n_0402, framos-csi-adapter-footprints:0402-cap, symbol framos-csi-adapter:C_100n_0402
- removed U2: NCP163ASN330T1G, framos-csi-adapter-footprints:SOT-23-5, symbol framos-csi-adapter:NCP163ASN330T1G
- added C? (x6): C_22u_0603, framos-csi-adapter-footprints:0603-cap, symbol framos-csi-adapter:C_22u_0603
- added C? (x8): C_100n_0402, framos-csi-adapter-footprints:0402-cap, symbol framos-csi-adapter:C_100n_0402
- added L?: XEL4030-332MEC, framos-csi-adapter-footprints:Coilcraft-XEL4030, symbol framos-csi-adapter:XEL4030-332MEC
- added L?: XEL4030-222MEC, framos-csi-adapter-footprints:Coilcraft-XEL4030, symbol framos-csi-adapter:XEL4030-222MEC
- added R?: R_14k7_0402, framos-csi-adapter-footprints:0402-res, symbol framos-csi-adapter:R_14k7_0402
- added R?: R_3k92_0402, framos-csi-adapter-footprints:0402-res, symbol framos-csi-adapter:R_3k92_0402
- added R?: R_12k4_0402, framos-csi-adapter-footprints:0402-res, symbol framos-csi-adapter:R_12k4_0402
- added R?: R_10k_0402, framos-csi-adapter-footprints:0402-res, symbol framos-csi-adapter:R_10k_0402
- added TP? (x2): TP_SMD1MM, framos-csi-adapter-footprints:Testpoint_smd_1mm, symbol framos-csi-adapter:TP_SMD1MM
- added U? (x2): AP62301Z6-7, framos-csi-adapter-footprints:SOT-563, symbol framos-csi-adapter:AP62301Z6-7
Connections:
- net labels added: 3V3FFC, 5V0_SYS
- net labels removed: 3V3
- wire segments 172 -> 218
- no-connect marks 15 -> 17
Other:
- note added: "1V8 MIPI Camera Power"
- note added: "3V8 MIPI Camera Power"
- note added: "EN - Active H\nEN float = auto startup"
- note removed: "3V3 LDO"
- moved on the sheet: C1, C2, D1, R11, R12, R2, U1

Commit message: Add 4-line CSI support - update pinout
Parts:
- added R? (x3): R_0R_0402, framos-csi-adapter-footprints:0402-res, symbol framos-csi-adapter:R_0R_0402
- added TP? (x7): TP_SMD_0_75MM, framos-csi-adapter-footprints:Testpoint_smd_0_75mm, symbol framos-csi-adapter:TP_SMD_0_75MM
- R10: DNP DNP -> (none)
Connections:
- net labels added: CSI_D2_N, CSI_D2_P, CSI_D3_N, CSI_D3_P
- wire segments 218 -> 247
- no-connect marks 17 -> 13
Other:
- note added: "Camera LED"
- note added: "Framos CSI interposer connector"
- note added: "I2C logic level translator bypass"
- note added: "JNB can have I2C configured as 1V8"
- note removed: "Host interface"
- moved on the sheet: C1, D1, R2

Commit message: Move power supply sections on PCB
Parts:
- removed C? (x2): C_100n_0402, framos-csi-adapter-footprints:0402-cap, symbol framos-csi-adapter:C_100n_0402
- removed TP?: TP_SMD1MM, framos-csi-adapter-footprints:Testpoint_smd_1mm, symbol framos-csi-adapter:TP_SMD1MM
- added TP6: TP_SMD_0_75MM, framos-csi-adapter-footprints:Testpoint_smd_0_75mm, symbol framos-csi-adapter:TP_SMD_0_75MM
- C10, C4: renamed from C?; footprint framos-csi-adapter-footprints:0402-cap -> antmicro-footprints:0402-cap; symbol framos-csi-adapter:C_100n_0402 -> antmicroCapacitors0402:C_100n_0402
- C13, C14, C3, C5, C6, C7: renamed from C?; footprint framos-csi-adapter-footprints:0603-cap -> antmicro-footprints:0603-cap; symbol framos-csi-adapter:C_22u_0603 -> antmicroCapacitors0603:C_22u_0603
- L1: renamed from L?; footprint framos-csi-adapter-footprints:Coilcraft-XEL4030 -> antmicro-footprints:Coilcraft-XEL4030; symbol framos-csi-adapter:XEL4030-332MEC -> antmicroFixedInductors:XEL4030-332MEC
- L2: renamed from L?; footprint framos-csi-adapter-footprints:Coilcraft-XEL4030 -> antmicro-footprints:Coilcraft-XEL4030; symbol framos-csi-adapter:XEL4030-222MEC -> antmicroFixedInductors:XEL4030-222MEC
- R14: renamed from R?; footprint framos-csi-adapter-footprints:0402-res -> antmicro-footprints:0402-res; symbol framos-csi-adapter:R_14k7_0402 -> antmicroResistors0402:R_14k7_0402
- R15: renamed from R?; footprint framos-csi-adapter-footprints:0402-res -> antmicro-footprints:0402-res; symbol framos-csi-adapter:R_3k92_0402 -> antmicroResistors0402:R_3k92_0402
- R16, R17: renamed from R?; footprint framos-csi-adapter-footprints:0402-res -> antmicro-footprints:0402-res; symbol framos-csi-adapter:R_0R_0402 -> antmicroResistors0402:R_0R_0402
- R18: renamed from R?; footprint framos-csi-adapter-footprints:0402-res -> antmicro-footprints:0402-res; symbol framos-csi-adapter:R_12k4_0402 -> antmicroResistors0402:R_12k4_0402
- R19: renamed from R?; footprint framos-csi-adapter-footprints:0402-res -> antmicro-footprints:0402-res; symbol framos-csi-adapter:R_10k_0402 -> antmicroResistors0402:R_10k_0402
- TP18: renamed from TP?; footprint framos-csi-adapter-footprints:Testpoint_smd_1mm -> antmicro-footprints:Testpoint_smd_1mm; symbol framos-csi-adapter:TP_SMD1MM -> antmicroTestPoints:TP_SMD1MM
- U2, U3: renamed from U?; footprint framos-csi-adapter-footprints:SOT-563 -> antmicro-footprints:SOT-563; symbol framos-csi-adapter:AP62301Z6-7 -> antmicroDCDCConverters:AP62301Z6-7
- gave numbers to parts that had none: 12
Connections:
- wire segments 247 -> 243
Other:
- moved on the sheet: C12

Commit message: Tweak FB resistors, change L1 and L2 to smaller size
Parts:
- removed L1: XEL4030-332MEC, antmicro-footprints:Coilcraft-XEL4030, symbol antmicroFixedInductors:XEL4030-332MEC
- removed L2: XEL4030-222MEC, antmicro-footprints:Coilcraft-XEL4030, symbol antmicroFixedInductors:XEL4030-222MEC
- removed R14: R_14k7_0402, antmicro-footprints:0402-res, symbol antmicroResistors0402:R_14k7_0402
- removed R15: R_3k92_0402, antmicro-footprints:0402-res, symbol antmicroResistors0402:R_3k92_0402
- added L1, L2: 74479887222C, framos-csi-adapter-footprints:L_1008_2520Metric, symbol framos-csi-adapter:74479887222C
- added R14: R_37k4_0402, framos-csi-adapter-footprints:0402-res, symbol framos-csi-adapter:R_37k4_0402
- added R15: R_10k_0402, framos-csi-adapter-footprints:0402-res, symbol framos-csi-adapter:R_10k_0402
- C10, C4: footprint antmicro-footprints:0402-cap -> framos-csi-adapter-footprints:0402-cap; symbol antmicroCapacitors0402:C_100n_0402 -> framos-csi-adapter:C_100n_0402
- C13, C14, C3, C5, C6, C7: footprint antmicro-footprints:0603-cap -> framos-csi-adapter-footprints:0603-cap; symbol antmicroCapacitors0603:C_22u_0603 -> framos-csi-adapter:C_22u_0603
- R16, R17: footprint antmicro-footprints:0402-res -> framos-csi-adapter-footprints:0402-res; symbol antmicroResistors0402:R_0R_0402 -> framos-csi-adapter:R_0R_0402
- R18: footprint antmicro-footprints:0402-res -> framos-csi-adapter-footprints:0402-res; symbol antmicroResistors0402:R_12k4_0402 -> framos-csi-adapter:R_12k4_0402
- R19: footprint antmicro-footprints:0402-res -> framos-csi-adapter-footprints:0402-res; symbol antmicroResistors0402:R_10k_0402 -> framos-csi-adapter:R_10k_0402
- TP18: footprint antmicro-footprints:Testpoint_smd_1mm -> framos-csi-adapter-footprints:Testpoint_smd_1mm; symbol antmicroTestPoints:TP_SMD1MM -> framos-csi-adapter:TP_SMD1MM
- U2, U3: footprint antmicro-footprints:SOT-563 -> framos-csi-adapter-footprints:SOT-563; symbol antmicroDCDCConverters:AP62301Z6-7 -> framos-csi-adapter:AP62301Z6-7

Commit message: Changed voltage translator to XSON8 package. Crossed P and N signals on D2 and D3 lanes
Parts:
- removed U1: NTS0102DP, framos-csi-adapter-footprints:TSSOP-8_W3mm, symbol framos-csi-adapter:NTS0102DP
- added U1: NTS0102GT, antmicro-footprints:PSON50P100X195X50-8N, symbol framos-csi-adapter:NTS0102GT
- R10, R9: DNP (none) -> DNP
Connections:
- wire segments 243 -> 245
Other:
- note added: "Pull-up resistors from 3V3 side are placed on JNB"
- moved on the sheet: TP17, TP18, TP19
Changed lines of the file:
@@
 F 5 "ERJ2GE0R00X" H 3050 4275 60  0001 L CNN "MPN"
 F 6 "0R" H 3000 3925 50  0000 C CNN "Val"
+F 7 "DNP" H 2850 3975 50  0000 C CNN "DNP"
 	1    2850 3975
 	1    0    0    -1
@@
 F 5 "ERJ2GE0R00X" H 3050 4375 60  0001 L CNN "MPN"
 F 6 "0R" H 3000 4025 50  0000 C CNN "Val"
+F 7 "DNP" H 2850 4075 50  0000 C CNN "DNP"
 	1    2850 4075
 	1    0    0    -1
@@
 	0    1    1    0
 $EndComp
-$Comp
-L framos-csi-adapter:NTS0102DP U1
-U 1 1 61D1A7EF
-P 6125 7750
-F 0 "U1" H 5875 8150 50  0000 C CNN
-F 1 "NTS0102DP" H 6125 7550 50  0000 C CNN
-F 2 "framos-csi-adapter-footprints:TSSOP-8_W3mm" H 6025 8250 50  0001 C CNN
-F 3 "" H 6775 8500 50  0001 C CNN
-F 4 "NTS0102DP" H 6075 7350 50  0001 C CNN "MPN"
-F 5 "NXP Semiconductors" H 6225 7450 50  0001 C CNN "Manufacturer"
-	1    6125 7750
-	1    0    0    -1
-$EndComp
 Text GLabel 4500 7600 0    50   BiDi ~ 0
 CAM_SCL_1V8
@@
 L framos-csi-adapter:TP_SMD1MM TP18
 U 1 1 622E82D8
-P 7975 9725
-F 0 "TP18" H 7925 9772 50  0000 R CNN
-F 1 "TP_SMD1MM" H 7975 9625 50  0001 C CNN
-F 2 "framos-csi-adapter-footprints:Testpoint_smd_1mm" H 8175 9925 60  0001 L CNN
-F 3 "" H 8175 10025 60  0001 L CNN
-	1    7975 9725
+P 7900 9725
+F 0 "TP18" H 7850 9772 50  0000 R CNN
+F 1 "TP_SMD1MM" H 7900 9625 50  0001 C CNN
+F 2 "framos-csi-adapter-footprints:Testpoint_smd_1mm" H 8100 9925 60  0001 L CNN
+F 3 "" H 8100 10025 60  0001 L CNN
+	1    7900 9725
 	-1   0    0    1
 $EndComp
 Wire Wire Line
-	8150 9825 7975 9825
-Connection ~ 7975 9825
+	8150 9825 7900 9825
+Connection ~ 7900 9825
 Wire Wire Line
-	7875 9825 7975 9825
+	7800 9825 7900 9825
 $Comp
 L framos-csi-adapter:C_100n_0402 C10
@@
 Text Notes 8250 10300 0    50   ~ 0
 EN - Active H\nEN float = auto startup
-NoConn ~ 7875 9825
+NoConn ~ 7800 9825
 $Comp
 L framos-csi-adapter:R_12k4_0402 R18
@@
 Text GLabel 8675 4800 1    50   Input ~ 0
 3V8_CAM
-Text GLabel 1925 4975 0    50   BiDi ~ 0
-CSI_D2_P
 Text GLabel 1925 4875 0    50   BiDi ~ 0
+CSI_D2_P
+Text GLabel 1925 4975 0    50   BiDi ~ 0
 CSI_D2_N
 Wire Wire Line
@@
 Wire Wire Line
 	1925 4875 3675 4875
-Text GLabel 6750 4275 2    50   BiDi ~ 0
-CSI_D3_N
 Text GLabel 6750 4375 2    50   BiDi ~ 0
+CSI_D3_N
+Text GLabel 6750 4275 2    50   BiDi ~ 0
 CSI_D3_P
 Wire Wire Line
@@
 L framos-csi-adapter:TP_SMD_0_75MM TP19
 U 1 1 6234F9CE
-P 10675 9525
-F 0 "TP19" V 10675 9400 50  0000 C CNN
-F 1 "TP_SMD_0_75MM" H 10675 9425 50  0001 C CNN
-F 2 "framos-csi-adapter-footprints:Testpoint_smd_0_75mm" H 10875 9725 60  0001 L CNN
-F 3 "" H 10875 9825 60  0001 L CNN
-	1    10675 9525
+P 10675 9475
+F 0 "TP19" H 10625 9522 50  0000 R CNN
+F 1 "TP_SMD_0_75MM" H 10675 9375 50  0001 C CNN
+F 2 "framos-csi-adapter-footprints:Testpoint_smd_0_75mm" H 10875 9675 60  0001 L CNN
+F 3 "" H 10875 9775 60  0001 L CNN
+	1    10675 9475
 	-1   0    0    1
 $EndComp
@@
 L framos-csi-adapter:TP_SMD_0_75MM TP17
 U 1 1 62352199
-P 4600 9600
-F 0 "TP17" H 4600 9525 50  0000 C CNN
-F 1 "TP_SMD_0_75MM" H 4600 9500 50  0001 C CNN
-F 2 "framos-csi-adapter-footprints:Testpoint_smd_0_75mm" H 4800 9800 60  0001 L CNN
-F 3 "" H 4800 9900 60  0001 L CNN
-	1    4600 9600
+P 4600 9550
+F 0 "TP17" H 4550 9597 50  0000 R CNN
+F 1 "TP_SMD_0_75MM" H 4600 9450 50  0001 C CNN
+F 2 "framos-csi-adapter-footprints:Testpoint_smd_0_75mm" H 4800 9750 60  0001 L CNN
+F 3 "" H 4800 9850 60  0001 L CNN
+	1    4600 9550
 	-1   0    0    1
 $EndComp
@@
 Wire Wire Line
 	2475 3275 3675 3275
-Text Notes 5025 6625 0    50   ~ 0
-JNB can have I2C configured as 1V8
 $Comp
 L framos-csi-adapter:R_0R_0402 R17
@@
 	0    1    1    0
 $EndComp
+Text Notes 7550 7675 0    50   ~ 0
+Pull-up resistors from 3V3 side are placed on JNB
+$Comp
+L framos-csi-adapter:NTS0102GT U1
+U 1 1 62CC3337
+P 6125 7750
+F 0 "U1" H 6125 8265 50  0000 C CNN
+F 1 "NTS0102GT" H 6125 8174 50  0000 C CNN
+F 2 "antmicro-footprints:PSON50P100X195X50-8N" H 6025 8250 50  0001 C CNN
+F 3 "http://www.farnell.com/datasheets/1760723.pdf" H 6775 8500 50  0001 C CNN
+F 4 "NTS0102GT" H 6125 8265 50  0001 C CNN "MPN"
+F 5 "NXP Semiconductors" H 6125 8174 50  0001 C CNN "Manufacturer"
+	1    6125 7750
+	1    0    0    -1
+$EndComp
+Wire Wire Line
+	10675 9575 10675 9625
+Wire Wire Line
+	4600 9650 4600 9700
 $EndSCHEMATC
